File: Hardware/Angra_v.1.0/Angra_v.1.0.sch (EAGLE design)
At the start: 88 parts, among them IC10 ESP32-WROOM-32U_M113DH2800UH3Q, IC11 TLV803EA30DCKR, IC12 FT232RL-REEL, IC2 MAX17201G+T, IC3 LM1117DT-3.3_NOPB, IC4 LT3652HVEMSE#PBF, IC5 LM234DT, IC6 TPS61092RSAR, IC7 TLV809ED29DBZR, IC8 TCAN330DR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

Commit message: Add files via upload
Other:
- note added: "1/1"
- note added: "C:/Users/marcu/Desktop/Ensino Superior/Graduação - Eng Elétrica/Zenith/zenith-v2.bmp"
- note added: "EESC - USP"
- note added: "João M. E. Morais A."
- note added: "Setembro de 2021"
- moved on the sheet: BT1, BT2, BT3, BT4, BT5, BT6, BT7, C10, C11, C12, C16, C17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
